Commit message: Added GPS

File: src/elsa_gazebo/urdf/elsa.xacro (robot description, xacro)
@@ -22,4 +22,6 @@
 <xacro:property name="lidar_mass" value="0"/>
 <xacro:property name="lidar_angle" value="0"/>
+<xacro:property name="gps_size" value="0.05"/>
+<xacro:property name="gps_mass" value="0"/>
 <xacro:include filename="$(find elsa_gazebo)/urdf/elsa.gazebo" />
 <xacro:include filename="$(find elsa_gazebo)/urdf/materials.xacro" />
