Commit message: New Robot Model
- Generalized the launch file system to work for multiple robots
- Created a new robot (temporarily named "Oaken") with a model more
  reflective of the new robot design, (2 wheel drive, caster wheels in
  the back), and the appropriate differential drive controller

File: src/sb_gazebo/urdf/elsa.xacro (robot description, xacro)
@@ -1,3 +1,6 @@
 <?xml version="1.0"?>
+<!--
+     The Model for Elsa, a 4-wheel drive, skid-steering robot
+-->
 <robot name="elsa" xmlns:xacro="http://www.ros.org/wiki/xacro">
 <xacro:property name="PI" value="3.1415926535897931"/>
@@ -24,7 +27,7 @@
 <xacro:property name="gps_size" value="0.05"/>
 <xacro:property name="gps_mass" value="0"/>
-<xacro:include filename="$(find elsa_gazebo)/urdf/elsa.gazebo" />
-<xacro:include filename="$(find elsa_gazebo)/urdf/materials.xacro" />
-<xacro:include filename="$(find elsa_gazebo)/urdf/macros.xacro" />
+<xacro:include filename="$(find sb_gazebo)/urdf/elsa.gazebo" />
+<xacro:include filename="$(find sb_gazebo)/urdf/materials.xacro" />
+<xacro:include filename="$(find sb_gazebo)/urdf/macros.xacro" />
 <!-- Footprint of the robot (because gazebo's base_link can't have interia) -->
 <link name='base_link'/>

File: src/sb_gazebo/urdf/macros.xacro (robot description, xacro)
@@ -1,3 +1,6 @@
 <?xml version="1.0"?>
+<!--
+    A Useful set of macros, mostly for generating model parts
+-->
 <robot name="elsa" xmlns:xacro="http://www.ros.org/wiki/xacro">
 <xacro:macro name="cylinder_inertia" params="m r h">
@@ -69,4 +72,56 @@
 </transmission>
 </xacro:macro>
+<!-- Macro to generate caster wheels -->
+<xacro:macro name="caster_wheel" params="lr tY wheel_displacement fb">
+<link name="${lr}_${fb}_wheel">
+  <collision>
+    <origin xyz="0 0 0" rpy="0 ${PI/2} ${PI/2}" />
+    <geometry>
+      <sphere radius="${wheel_radius}"/>
+    </geometry>
+  </collision>
+  <visual>
+    <origin xyz="0 0 0" rpy="0 ${PI/2} ${PI/2}" />
+    <geometry>
+      <sphere radius="${wheel_radius}"/>
+    </geometry>
+    <material name="black"/>
+  </visual>
+  <inertial>
+    <origin xyz="0 0 0" rpy="0 ${PI/2} ${PI/2}" />
+    <mass value="${wheel_mass}"/>
+    <sphere_inertia m="${wheel_mass}" r="${wheel_radius}"/>
+  </inertial>
+</link>
+<gazebo reference="${lr}_${fb}_wheel">
+  <mu1 value="1.0"/>
+  <mu2 value="1.0"/>
+  <kp  value="10000000.0" />
+  <kd  value="1.0" />
+  <fdir1 value="1 0 0"/>
+  <material>Gazebo/Black</material>
+</gazebo>
+<joint name="${lr}_${fb}_wheel_hinge" type="continuous">
+  <parent link="chassis"/>
+  <child link="${lr}_${fb}_wheel"/>
+  <origin xyz="${wheel_displacement} ${-tY*wheel_width+tY*chassis_width/2} ${wheel_radius}" rpy="0 0 0" />
+  <axis xyz="0 1 0" rpy="0 0 0" />
+  <limit effort="100" velocity="100"/>
+  <joint_properties damping="1.0" friction="1.0"/>
+  <hardwareInterface>EffortJointInterface</hardwareInterface>
+</joint>
+<!--
+<transmission name="${lr}_${fb}_trans">
+  <type>transmission_interface/SimpleTransmission</type>
+  <joint name="${lr}_${fb}_wheel_hinge">
+    <hardwareInterface>EffortJointInterface</hardwareInterface>
+  </joint>
+  <actuator name="${lr}_${fb}_Motor">
+    <hardwareInterface>EffortJointInterface</hardwareInterface>
+    <mechanicalReduction>10</mechanicalReduction>
+  </actuator>
+</transmission>
+-->
+</xacro:macro>
 <!-- Macro to generate vertical tower uprights -->
 <xacro:macro name="tower_vert" params="lr tY">

File: src/sb_gazebo/urdf/materials.xacro (robot description, xacro)
@@ -1,3 +1,6 @@
 <?xml version="1.0"?>
+<!--
+     The Materials for all Robots
+ -->
 <robot name="elsa" xmlns:xacro="http://www.ros.org/wiki/xacro">
 <material name="black">
