Commit message: Updated robot dimensions

File: src/sb_gazebo/urdf/oaken.xacro (robot description, xacro)
@@ -5,6 +5,6 @@
 <robot name="oaken" xmlns:xacro="http://www.ros.org/wiki/xacro">
 <xacro:property name="PI" value="3.1415926535897931"/>
-<xacro:property name="chassis_length" value="0.85" />
-<xacro:property name="chassis_width" value="0.85" />
+<xacro:property name="chassis_length" value="0.91" />
+<xacro:property name="chassis_width" value="0.71" />
 <xacro:property name="chassis_height" value="0.35" />
 <xacro:property name="chassis_mass" value="30" />
