Commit message: fixed physics

File: src/sb_gazebo/urdf/macros.xacro (robot description, xacro)
@@ -3,5 +3,5 @@
     A Useful set of macros, mostly for generating model parts
 -->
-<robot name="elsa" xmlns:xacro="http://www.ros.org/wiki/xacro">
+<robot name="robot" xmlns:xacro="http://www.ros.org/wiki/xacro">
 <xacro:macro name="cylinder_inertia" params="m r h">
   <inertia  ixx="${m*(3*r*r+h*h)/12}" ixy = "0" ixz = "0"
@@ -45,6 +45,6 @@
 </link>
 <gazebo reference="${lr}_${fb}_wheel">
-  <mu1 value="1.0"/>
-  <mu2 value="1.0"/>
+  <mu1 value="10.0"/>
+  <mu2 value="10.0"/>
   <kp  value="10000000.0" />
   <kd  value="1.0" />
@@ -74,5 +74,5 @@
 <!-- Macro to generate caster wheels -->
 <xacro:macro name="caster_wheel" params="lr tY wheel_displacement fb">
-<link name="${lr}_${fb}_wheel">
+<link name="${lr}_${fb}_caster_wheel">
   <collision>
     <origin xyz="0 0 0" rpy="0 ${PI/2} ${PI/2}" />
@@ -80,4 +80,14 @@
       <sphere radius="${wheel_radius}"/>
     </geometry>
+    <surface>
+      <friction>
+        <ode>
+          <mu>0</mu>
+          <mu2>0</mu2>
+          <slip1>1</slip1>
+          <slip2>1</slip2>
+        </ode>
+      </friction>
+    </surface>
   </collision>
   <visual>
@@ -90,16 +100,14 @@
   <inertial>
     <origin xyz="0 0 0" rpy="0 ${PI/2} ${PI/2}" />
-    <mass value="${wheel_mass}"/>
-    <sphere_inertia m="${wheel_mass}" r="${wheel_radius}"/>
+    <mass value="0"/>
+    <sphere_inertia m="0" r="0"/>
   </inertial>
 </link>
-<gazebo reference="${lr}_${fb}_wheel">
-  <mu1 value="1.0"/>
-  <mu2 value="1.0"/>
-  <kp  value="10000000.0" />
-  <kd  value="1.0" />
-  <fdir1 value="1 0 0"/>
+<gazebo reference="${lr}_${fb}_caster_wheel">
+  <mu1 value="0.0"/>
+  <mu2 value="0.0"/>
   <material>Gazebo/Black</material>
 </gazebo>
+<!--
 <joint name="${lr}_${fb}_wheel_hinge" type="continuous">
   <parent link="chassis"/>
@@ -108,19 +116,13 @@
   <axis xyz="0 1 0" rpy="0 0 0" />
   <limit effort="100" velocity="100"/>
-  <joint_properties damping="1.0" friction="1.0"/>
+  <joint_properties damping="0.0" friction="0.0"/>
   <hardwareInterface>EffortJointInterface</hardwareInterface>
 </joint>
-<!--
-<transmission name="${lr}_${fb}_trans">
-  <type>transmission_interface/SimpleTransmission</type>
-  <joint name="${lr}_${fb}_wheel_hinge">
-    <hardwareInterface>EffortJointInterface</hardwareInterface>
-  </joint>
-  <actuator name="${lr}_${fb}_Motor">
-    <hardwareInterface>EffortJointInterface</hardwareInterface>
-    <mechanicalReduction>10</mechanicalReduction>
-  </actuator>
-</transmission>
 -->
+<joint name="${lr}_${fb}_wheel_hinge" type="fixed">
+  <parent link="chassis"/>
+  <child link="${lr}_${fb}_caster_wheel"/>
+  <origin xyz="${wheel_displacement} ${-tY*wheel_width+tY*chassis_width/2} ${wheel_radius}" rpy="0 0 0" />
+</joint>
 </xacro:macro>
 <!-- Macro to generate vertical tower uprights -->
