Commit message: updated tower placement

File: src/sb_gazebo/urdf/elsax.xacro (robot description, xacro)
@@ -66,6 +66,6 @@
   <caster_wheel lr="back" tY="0" fb="back" wheel_displacement="-0.35"/>
   <!-- Vertical Tower Uprights -->
-  <tower_vert lr="left" tY="1"/>
-  <tower_vert lr="right" tY="-1"/>
+  <tower_vert lr="left" tY="1" tX="1"/>
+  <tower_vert lr="right" tY="-1" tX="1"/>
   <!-- Horizontal Tower Top Bar -->
   <joint name="tower_top_bar_joint" type="fixed">
@@ -73,5 +73,5 @@
     <child link="tower_top_bar"/>
     <origin
-        xyz="${-(chassis_length/2) + (tower_thickness/2)} 0 ${chassis_height + chassis_elevation + tower_height - (tower_thickness/2)}"
+        xyz="${(chassis_length/2) - (tower_thickness/2)} 0 ${chassis_height + chassis_elevation + tower_height - (tower_thickness/2)}"
         rpy="0 0 0"/>
   </joint>
@@ -100,5 +100,5 @@
     <parent link="chassis"/>
     <child link="camera"/>
-    <origin xyz="${-(chassis_length/2)} 0 ${chassis_height + chassis_elevation + tower_height + camera_size}"
+    <origin xyz="${(chassis_length/2)} 0 ${chassis_height + chassis_elevation + tower_height + camera_size}"
             rpy="0 ${camera_angle} 0"/>
   </joint>

File: src/sb_gazebo/urdf/macros.xacro (robot description, xacro)
@@ -127,9 +127,9 @@
 </xacro:macro>
 <!-- Macro to generate vertical tower uprights -->
-<xacro:macro name="tower_vert" params="lr tY">
+<xacro:macro name="tower_vert" params="lr tX:=-1 tY">
 <joint name="${lr}_tower_joint" type="fixed">
   <parent link="chassis"/>
   <child link="tower_${lr}"/>
-  <origin xyz="${-(chassis_length/2) + (tower_thickness/2)} ${tY * ((chassis_width/2) - (tower_thickness/2))} ${chassis_height + chassis_elevation + (tower_height/2)}" rpy="0 0 0"/>
+  <origin xyz="${tX * ((chassis_length/2) - (tower_thickness/2))} ${tY * ((chassis_width/2) - (tower_thickness/2))} ${chassis_height + chassis_elevation + (tower_height/2)}" rpy="0 0 0"/>
 </joint>
 <link name='tower_${lr}'>

Commit message: updated wheel sizes

File: src/sb_gazebo/urdf/elsax.xacro (robot description, xacro)
@@ -12,8 +12,10 @@
   <xacro:property name="tower_thickness" value="0.05"/>
   <xacro:property name="tower_mass" value="0"/>
-  <xacro:property name="wheel_radius" value="0.10"/>
-  <xacro:property name="wheel_width" value="0.10"/>
+  <xacro:property name="wheel_radius" value="0.21"/>
+  <xacro:property name="wheel_width" value="0.12"/>
   <xacro:property name="wheel_displace" value="0.0"/>
   <xacro:property name="wheel_mass" value="1"/>
+  <xacro:property name="caster_radius" value="0.04" />
+  <xacro:property name="caster_mass" value="1"/>
   <xacro:property name="camera_size" value="0.05"/>
   <xacro:property name="camera_mass" value="0.1"/>
@@ -60,9 +62,6 @@
   <wheel lr="right" tY="-1" fb="centre" wheel_displacement="${wheel_displace}"/>
   <!-- Caster Wheels -->
-  <!--
-  <caster_wheel lr="left" tY="1" fb="back" wheel_displacement="${-wheel_displace}"/>
-  -->
-  <caster_wheel lr="front" tY="0" fb="front" wheel_displacement="0.35"/>
-  <caster_wheel lr="back" tY="0" fb="back" wheel_displacement="-0.35"/>
+  <caster_wheel lr="front" tY="0" fb="front" wheel_displacement="0.35" caster_radius="${caster_radius}"/>
+  <caster_wheel lr="back" tY="0" fb="back" wheel_displacement="-0.35" caster_radius="${caster_radius}"/>
   <!-- Vertical Tower Uprights -->
   <tower_vert lr="left" tY="1" tX="1"/>

File: src/sb_gazebo/urdf/macros.xacro (robot description, xacro)
@@ -73,10 +73,10 @@
 </xacro:macro>
 <!-- Macro to generate caster wheels -->
-<xacro:macro name="caster_wheel" params="lr tY wheel_displacement fb">
+<xacro:macro name="caster_wheel" params="lr tY wheel_displacement fb caster_radius:=${wheel_radius}">
 <link name="${lr}_${fb}_caster_wheel">
   <collision>
     <origin xyz="0 0 0" rpy="0 ${pi/2} ${pi/2}" />
     <geometry>
-      <sphere radius="${wheel_radius}"/>
+      <sphere radius="${caster_radius}"/>
     </geometry>
     <surface>
@@ -94,5 +94,5 @@
     <origin xyz="0 0 0" rpy="0 ${pi/2} ${pi/2}" />
     <geometry>
-      <sphere radius="${wheel_radius}"/>
+      <sphere radius="${caster_radius}"/>
     </geometry>
     <material name="black"/>
@@ -113,5 +113,5 @@
   <parent link="chassis"/>
   <child link="${lr}_${fb}_wheel"/>
-  <origin xyz="${wheel_displacement} ${-tY*wheel_width+tY*chassis_width/2} ${wheel_radius}" rpy="0 0 0" />
+  <origin xyz="${wheel_displacement} ${-tY*wheel_width+tY*chassis_width/2} ${caster_radius}" rpy="0 0 0" />
   <axis xyz="0 1 0" rpy="0 0 0" />
   <limit effort="100" velocity="100"/>
@@ -123,5 +123,5 @@
   <parent link="chassis"/>
   <child link="${lr}_${fb}_caster_wheel"/>
-  <origin xyz="${wheel_displacement} ${-tY*wheel_width+tY*chassis_width/2} ${wheel_radius}" rpy="0 0 0" />
+  <origin xyz="${wheel_displacement} ${-tY*caster_radius+tY*chassis_width/2} ${caster_radius}" rpy="0 0 0" />
 </joint>
 </xacro:macro>
