Commit message: Updating Rover Model To Be Xacro compatible

File: src/sb_gazebo/robots/rover_2018.xacro (robot description, xacro)
@@ -8,16 +8,22 @@
 -->
 <robot name="rover_2018" xmlns:xacro="http://www.ros.org/wiki/xacro">
+    <!-- Footprint of the robot (because gazebo's base_link can't have interia) -->
+    <link name='base_link'/>
+    <joint name="base_joint" type="fixed">
+        <parent link="base_link"/>
+        <child link="main_chassis"/>
+    </joint>
     <link name='main_chassis'>
         <pose frame=''>-0.495954 0.481744 0.172621 0 -0 0</pose>
         <inertial>
-            <mass>10</mass>
-            <inertia>
-                <ixx>0.01</ixx>
-                <ixy>0</ixy>
-                <ixz>0</ixz>
-                <iyy>0.01</iyy>
-                <iyz>0</iyz>
-                <izz>0.01</izz>
-            </inertia>
+            <mass value="10"/>
+            <inertia
+                ixx="0.01"
+                ixy="0"
+                ixz="0"
+                iyy="0.01"
+                iyz="0"
+                izz="0.01"
+            />
             <pose frame=''>0 0 0 0 -0 0</pose>
         </inertial>
@@ -28,9 +34,9 @@
             <pose frame=''>0 0 0 0 -0 0</pose>
             <geometry>
-                <box>
-                    <size>1.09569 1.7415 0.312322</size>
-                </box>
-            </geometry>
-            <material>
+                <box
+                    size="1.09569 1.7415 0.312322"
+                />
+            </geometry>
+            <material name="grey">
                 <lighting>1</lighting>
                 <script>
@@ -54,7 +60,7 @@
             <pose frame=''>0 0 0 0 -0 0</pose>
             <geometry>
-                <box>
-                    <size>1.09569 1.7415 0.312322</size>
-                </box>
+                <box
+                    size="1.09569 1.7415 0.312322"
+                />
             </geometry>
             <surface>
@@ -108,13 +114,13 @@
         <pose frame=''>0.120732 0.480291 0.210888 3.14159 -1.57 -3.14159</pose>
         <inertial>
-            <mass>0.0046174</mass>
-            <inertia>
-                <ixx>0.01</ixx>
-                <ixy>0</ixy>
-                <ixz>0</ixz>
-                <iyy>0.01</iyy>
-                <iyz>0</iyz>
-                <izz>0.01</izz>
-            </inertia>
+            <mass value="0.0046174"/>
+            <inertia
+                ixx="0.01"
+                ixy="0"
+                ixz="0"
+                iyy="0.01"
+                iyz="0"
+                izz="0.01"
+            />
             <pose frame=''>0 0 0 0 -0 0</pose>
         </inertial>
@@ -125,10 +131,10 @@
             <pose frame=''>0 0 0 0 -0 0</pose>
             <geometry>
-                <cylinder>
-                    <radius>0.0992866</radius>
-                    <length>0.116478</length>
-                </cylinder>
-            </geometry>
-            <material>
+                <cylinder
+                    radius="0.0992866"
+                    length="0.116478"
+                />
+            </geometry>
+            <material name="grey">
                 <lighting>1</lighting>
                 <script>
@@ -151,13 +157,13 @@
         <pose frame=''>0.045335 0.475634 0.210685 3.14159 -1.57 -3.14159</pose>
         <inertial>
-            <mass>0.00110726</mass>
-            <inertia>
-                <ixx>0.01</ixx>
-                <ixy>0</ixy>
-                <ixz>0</ixz>
-                <iyy>0.01</iyy>
-                <iyz>0</iyz>
-                <izz>0.01</izz>
-            </inertia>
+            <mass value="0.00110726"/>
+            <inertia
+                ixx="0.01"
+                ixy="0"
+                ixz="0"
+                iyy="0.01"
+                iyz="0"
+                izz="0.01"
+            />
             <pose frame=''>0 0 0 0 -0 0</pose>
         </inertial>
@@ -168,10 +174,10 @@
             <pose frame=''>0 0 0 0 -0 0</pose>
             <geometry>
-                <cylinder>
-                    <radius>0.0379471</radius>
-                    <length>0.191181</length>
-                </cylinder>
-            </geometry>
-            <material>
+                <cylinder
+                    radius="0.0379471"
+                    length="0.191181"
+                />
+            </geometry>
+            <material name="grey">
                 <lighting>1</lighting>
                 <script>
@@ -194,13 +200,13 @@
         <pose frame=''>0.120732 0.773902 0.074463 -0.422885 0 0</pose>
         <inertial>
-            <mass>0.00541225</mass>
-            <inertia>
-                <ixx>0.01</ixx>
-                <ixy>0</ixy>
-                <ixz>0</ixz>
-                <iyy>0.01</iyy>
-                <iyz>0</iyz>
-                <izz>0.01</izz>
-            </inertia>
+            <mass value="0.00541225"/>
+            <inertia
+                ixx="0.01"
+                ixy="0"
+                ixz="0"
+                iyy="0.01"
+                iyz="0"
+                izz="0.01"
+            />
             <pose frame=''>0 0 0 0 -0 0</pose>
         </inertial>
@@ -212,9 +218,9 @@
             <pose frame=''>0 0 0 0 -0 0</pose>
             <geometry>
-                <box>
-                    <size>0.093481 0.512407 0.11302</size>
-                </box>
-            </geometry>
-            <material>
+                <box
+                    size="0.093481 0.512407 0.11302"
+                />
+            </geometry>
+            <material name="grey">
                 <lighting>1</lighting>
                 <script>
@@ -238,7 +244,7 @@
             <pose frame=''>0 0 0 0 -0 0</pose>
             <geometry>
-                <box>
-                    <size>0.093481 0.512407 0.11302</size>
-                </box>
+                <box
+                    size="0.093481 0.512407 0.11302"
+                />
             </geometry>
             <surface>
@@ -292,13 +298,13 @@
         <pose frame=''>0.120732 0.030921 0.003788 0.410827 -0 0</pose>
         <inertial>
-            <mass>0.00955178</mass>
-            <inertia>
-                <ixx>0.01</ixx>
-                <ixy>0</ixy>
-                <ixz>0</ixz>
-                <iyy>0.01</iyy>
-                <iyz>0</iyz>
-                <izz>0.01</izz>
-            </inertia>
+            <mass value="0.00955178"/>
+            <inertia
+                ixx="0.01"
+                ixy="0"
+                ixz="0"
+                iyy="0.01"
+                iyz="0"
+                izz="0.01"
+            />
             <pose frame=''>0 0 0 0 -0 0</pose>
         </inertial>
@@ -309,9 +315,9 @@
             <pose frame=''>0 0 0 0 -0 0</pose>
             <geometry>
-                <box>
-                    <size>0.093481 0.904318 0.11302</size>
-                </box>
-            </geometry>
-            <material>
+                <box
+                    size="0.093481 0.904318 0.11302"
+                />
+            </geometry>
+            <material name="grey">
                 <lighting>1</lighting>
                 <script>
@@ -335,7 +341,7 @@
             <pose frame=''>0 0 0 0 -0 0</pose>
             <geometry>
-                <box>
-                    <size>0.093481 0.904318 0.11302</size>
-                </box>
+                <box
+                    size="0.093481 0.904318 0.11302"
+                />
             </geometry>
             <surface>
@@ -389,13 +395,13 @@
         <pose frame=''>0.227534 0.930061 -0.012476 3.14159 -1.57 -3.14159</pose>
         <inertial>
-            <mass>0.00158531</mass>
-            <inertia>
-                <ixx>0.01</ixx>
-                <ixy>0</ixy>
-                <ixz>0</ixz>
-                <iyy>0.01</iyy>
-                <iyz>0</iyz>
-                <izz>0.01</izz>
-            </inertia>
+            <mass value="0.00158531"/>
+            <inertia
+                ixx="0.01"
+                ixy="0"
+                ixz="0"
+                iyy="0.01"
+                iyz="0"
+                izz="0.01"
+            />
             <pose frame=''>0 0 0 0 -0 0</pose>
         </inertial>
@@ -407,10 +413,10 @@
             <pose frame=''>0 0 0 0 -0 0</pose>
             <geometry>
-                <cylinder>
-                    <radius>0.0665773</radius>
-                    <length>0.088915</length>
-                </cylinder>
-            </geometry>
-            <material>
+                <cylinder
+                    radius="0.0665773"
+                    length="0.088915"
+                />
+            </geometry>
+            <material name="grey">
                 <lighting>1</lighting>
                 <script>
@@ -433,13 +439,13 @@
         <pose frame=''>0.173471 0.937461 -0.010085 3.14159 -1.57 -3.14159</pose>
         <inertial>
-            <mass>0.00016166</mass>
-            <inertia>
-                <ixx>0.01</ixx>
-                <ixy>0</ixy>
-                <ixz>0</ixz>
-                <iyy>0.01</iyy>
-                <iyz>0</iyz>
-                <izz>0.01</izz>
-            </inertia>
+            <mass value="0.00016166"/>
+            <inertia
+                ixx="0.01"
+                ixy="0"
+                ixz="0"
+                iyy="0.01"
+                iyz="0"
+                izz="0.01"
+            />
             <pose frame=''>0 0 0 0 -0 0</pose>
         </inertial>
@@ -451,10 +457,10 @@
             <pose frame=''>0 0 0 0 -0 0</pose>
             <geometry>
-                <cylinder>
-                    <radius>0.0152481</radius>
-                    <length>0.138038</length>
-                </cylinder>
-            </geometry>
-            <material>
+                <cylinder
+                    radius="0.0152481"
+                    length="0.138038"
+                />
+            </geometry>
+            <material name="grey">
                 <lighting>1</lighting>
                 <script>
@@ -477,13 +483,13 @@
         <pose frame=''>0.227534 1.14505 -0.096467 -0.359364 0 0</pose>
         <inertial>
-            <mass>0.0019482</mass>
-            <inertia>
-                <ixx>0.01</ixx>
-                <ixy>0</ixy>
-                <ixz>0</ixz>
-                <iyy>0.01</iyy>
-                <iyz>0</iyz>
-                <izz>0.01</izz>
-            </inertia>
+            <mass value="0.0019482"/>
+            <inertia
+                ixx="0.01"
+                ixy="0"
+                ixz="0"
+                iyy="0.01"
+                iyz="0"
+                izz="0.01"
+            />
             <pose frame=''>0 0 0 0 -0 0</pose>
         </inertial>
@@ -494,9 +500,9 @@
             <pose frame=''>0 0 0 0 -0 0</pose>
             <geometry>
-                <box>
-                    <size>0.062968 0.419703 0.073703</size>
-                </box>
-            </geometry>
-            <material>
+                <box
+                    size="0.062968 0.419703 0.073703"
+                />
+            </geometry>
+            <material name="grey">
                 <lighting>1</lighting>
                 <script>
@@ -518,7 +524,7 @@
             <pose frame=''>0 0 0 0 -0 0</pose>
             <geometry>
-                <box>
-                    <size>0.062968 0.419703 0.073703</size>
-                </box>
+                <box
+                    size="0.062968 0.419703 0.073703"
+                />
             </geometry>
             <surface>
@@ -572,13 +578,13 @@
         <pose frame=''>0.227534 0.747337 -0.096816 0.366679 -0 0</pose>
         <inertial>
-            <mass>0.00190054</mass>
-            <inertia>
-                <ixx>0.01</ixx>
-                <ixy>0</ixy>
-                <ixz>0</ixz>
-                <iyy>0.01</iyy>
-                <iyz>0</iyz>
-                <izz>0.01</izz>
-            </inertia>
+            <mass value="0.00190054"/>
+            <inertia
+                ixx="0.01"
+                ixy="0"
+                ixz="0"
+                iyy="0.01"
+                iyz="0"
+                izz="0.01"
+            />
             <pose frame=''>0 0 0 0 -0 0</pose>
         </inertial>
@@ -589,9 +595,9 @@
             <pose frame=''>0 0 0 0 -0 0</pose>
             <geometry>
-                <box>
-                    <size>0.062968 0.40946 0.073703</size>
-                </box>
-            </geometry>
-            <material>
+                <box
+                    size="0.062968 0.40946 0.073703"
+                />
+            </geometry>
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
Commit message: Revised Rover Model To Use Relative Positions

File: src/sb_gazebo/robots/rover_2018.xacro (robot description, xacro)
@@ -24,17 +24,19 @@
     <xacro:property name="primary_rocker_arm_radius" value="0.03"/>
     <xacro:property name="primary_rocker_arm_pitch" value="${pi*2.7/4}"/>
-    <xacro:property name="primary_rocker_arm_x_pos" value="${primary_rocker_x_pos}"/>
-    <xacro:property name="primary_rocker_arm_y_pos" value="${primary_rocker_radius - cos(primary_rocker_arm_pitch)*primary_rocker_arm_length/2}"/>
-    <xacro:property name="primary_rocker_arm_z_pos" value="${chassis_z_size + chassis_elevation - sin(primary_rocker_arm_pitch)*primary_rocker_arm_length/2}"/>
+    <xacro:property name="primary_rocker_arm_x_offset" value="0"/>
+    <xacro:property name="primary_rocker_arm_y_offset" value="${primary_rocker_radius - cos(primary_rocker_arm_pitch)*primary_rocker_arm_length/2}"/>
+    <xacro:property name="primary_rocker_arm_z_offset" value="${- sin(primary_rocker_arm_pitch)*primary_rocker_arm_length/2}"/>
     <xacro:property name="primary_wheel_axle_length" value="0.1"/>
     <xacro:property name="primary_wheel_axle_radius" value="0.015"/>
-    <xacro:property name="primary_wheel_axle_x_pos" value="${primary_rocker_x_pos}"/>
-    <xacro:property name="primary_wheel_axle_y_pos" value="${primary_rocker_y_pos + cos(primary_rocker_arm_pitch)*primary_rocker_arm_length*2}"/>
-    <xacro:property name="primary_wheel_axle_z_pos" value="${primary_rocker_arm_z_pos - sin(primary_rocker_arm_pitch)*primary_rocker_arm_length/2}"/>
+    <xacro:property name="primary_wheel_axle_x_offset" value="${primary_wheel_axle_length/2}"/>
+    <xacro:property name="primary_wheel_axle_y_offset"
+        value="${sin(primary_rocker_arm_pitch)*primary_rocker_arm_length/2}"/>
+    <xacro:property name="primary_wheel_axle_z_offset"
+        value="${cos(primary_rocker_arm_pitch)*primary_rocker_arm_length/2}"/>
     <xacro:property name="primary_wheel_length" value="0.15"/>
     <xacro:property name="primary_wheel_radius" value="0.17"/>
-    <xacro:property name="primary_wheel_x_pos" value="${primary_wheel_axle_x_pos + primary_wheel_axle_length/2 + primary_wheel_length/2}"/>
-    <xacro:property name="primary_wheel_y_pos" value="${primary_wheel_axle_y_pos}"/>
-    <xacro:property name="primary_wheel_z_pos" value="${primary_wheel_axle_z_pos}"/>
+    <xacro:property name="primary_wheel_x_offset" value="${primary_wheel_length/2}"/>
+    <xacro:property name="primary_wheel_y_offset" value="0"/>
+    <xacro:property name="primary_wheel_z_offset" value="0"/>
     <!-- Footprint of the robot (because gazebo's base_link can't have interia) -->
     <link name='base_link'/>
@@ -58,13 +60,19 @@
         />
     <xacro:macro name="primary_rocker" params="lr_prefix reflect">
-        <joint name="${lr_prefix}_primary_rocker_to_chassis" type="fixed">
+        <!-- TODO: Make this revolute model with a spring to resist rotation (but allow it) instead of just being fixed like it currently is -->
+        <joint name="${lr_prefix}_primary_rocker_to_chassis" type="revolute">
             <parent link="chassis"/>
             <child link="${lr_prefix}_primary_rocker"/>
+            <origin xyz="${primary_rocker_x_pos*reflect} ${primary_rocker_y_pos} ${primary_rocker_z_pos}" rpy="0 0 0" />
+            <axis xyz="1 0 0" rpy="0 0 0" />
+            <limit effort="100" velocity="100"/>
+            <joint_properties damping="0.0" friction="0.0"/>
+            <limit lower="-20" upper="20" effort="100" velocity="100"/>
         </joint>
         <cylinder_link
             name="${lr_prefix}_primary_rocker"
-            x_pos="${primary_rocker_x_pos*reflect}"
-            y_pos="${primary_rocker_y_pos}"
-            z_pos="${primary_rocker_z_pos}"
+            x_pos="0"
+            y_pos="0"
+            z_pos="0"
             radius="${primary_rocker_radius}"
             length="${primary_rocker_length}"
@@ -82,10 +90,17 @@
             <parent link="${lr_prefix}_primary_rocker"/>
             <child link="${lr_prefix}_${fb_prefix}_primary_rocker_arm"/>
+            <origin xyz="
+                ${primary_rocker_arm_x_offset*x_reflect}
+                ${primary_rocker_arm_y_offset*y_reflect}
+                ${primary_rocker_arm_z_offset}
+                "
+                rpy="0 0 0"
+            />
         </joint>
         <cylinder_link
             name="${lr_prefix}_${fb_prefix}_primary_rocker_arm"
-            x_pos="${primary_rocker_arm_x_pos*x_reflect}"
-            y_pos="${primary_rocker_arm_y_pos*y_reflect}"
-            z_pos="${primary_rocker_arm_z_pos}"
+            x_pos="0"
+            y_pos="0"
+            z_pos="0"
             radius="${primary_rocker_arm_radius}"
             length="${primary_rocker_arm_length}"
@@ -105,10 +120,17 @@
             <parent link="${lr_prefix}_${fb_prefix}_primary_rocker_arm"/>
             <child link="${lr_prefix}_${fb_prefix}_primary_wheel_axle"/>
+            <origin xyz="
+                ${primary_wheel_axle_x_offset*x_reflect}
+                ${primary_wheel_axle_y_offset*y_reflect}
+                ${primary_wheel_axle_z_offset}
+                "
+                rpy="0 0 0"
+            />
         </joint>
         <cylinder_link
             name="${lr_prefix}_${fb_prefix}_primary_wheel_axle"
-            x_pos="${(primary_wheel_axle_x_pos + primary_wheel_axle_length/2)*x_reflect}"
-            y_pos="${primary_wheel_axle_y_pos*y_reflect}"
-            z_pos="${primary_wheel_axle_z_pos}"
+            x_pos="0"
+            y_pos="0"
+            z_pos="0"
             radius="${primary_wheel_axle_radius}"
             length="${primary_wheel_axle_length}"
@@ -126,7 +148,13 @@
     <xacro:macro name="primary_wheel" params="lr_prefix fb_prefix x_reflect y_reflect">
         <joint name="${lr_prefix}_${fb_prefix}_primary_rocker_arm_to_primary_wheel" type="continuous">
-            <parent link="${lr_prefix}_${fb_prefix}_primary_rocker_arm"/>
+            <parent link="${lr_prefix}_${fb_prefix}_primary_wheel_axle"/>
             <child link="${lr_prefix}_${fb_prefix}_primary_wheel"/>
-            <origin xyz="${primary_wheel_x_pos*x_reflect} ${primary_wheel_y_pos*y_reflect} ${primary_wheel_z_pos}" rpy="0 0 0" />
+            <origin xyz="
+                ${primary_wheel_x_offset*x_reflect}
+                ${primary_wheel_y_offset*y_reflect}
+                ${primary_wheel_z_offset}
+                "
+                rpy="0 0 0"
+                />
             <axis xyz="1 0 0" rpy="0 0 0" />
             <limit effort="100" velocity="100"/>
