Commit message: Added Tower And Camera To Rover 2018 Model

File: src/sb_gazebo/robots/rover_2018.xacro (robot description, xacro)
@@ -1,7 +1,11 @@
 <?xml version="1.0"?>
 <!--
-     The Model for elsa-x, a 2-wheel drive robot with front and back caster wheels
+     The model for the 2018 rover
 -->
 <robot name="rover_2018" xmlns:xacro="http://www.ros.org/wiki/xacro">
+    <!-- CALCULATIONS
+         This section holds all the math to calculate the offset (both linear
+         and angular) for various components.
+    -->
     <xacro:include filename="$(find sb_gazebo)/robots/macros.xacro"/>
     <xacro:include filename="$(find sb_gazebo)/robots/materials.xacro"/>
@@ -18,7 +22,7 @@
     <xacro:property name="primary_rocker_length" value="0.1"/>
     <xacro:property name="primary_rocker_chassis_clearance" value="0.1"/>
-    <xacro:property name="primary_rocker_x_pos" value="${chassis_x_size/2 + primary_rocker_length/2 + primary_rocker_chassis_clearance}"/>
-    <xacro:property name="primary_rocker_y_pos" value="0"/>
-    <xacro:property name="primary_rocker_z_pos" value="${chassis_z_size + chassis_elevation}"/>
+    <xacro:property name="primary_rocker_x_offset" value="${chassis_x_size/2 + primary_rocker_length/2 + primary_rocker_chassis_clearance}"/>
+    <xacro:property name="primary_rocker_y_offset" value="0"/>
+    <xacro:property name="primary_rocker_z_offset" value="0"/>
     <xacro:property name="primary_rocker_arm_length" value="0.4"/>
     <xacro:property name="primary_rocker_arm_radius" value="0.03"/>
@@ -39,4 +43,17 @@
     <xacro:property name="primary_wheel_y_offset" value="0"/>
     <xacro:property name="primary_wheel_z_offset" value="0"/>
+    <xacro:property name="tower_upright_y_offset" value="${chassis_y_size/2}"/>
+    <xacro:property name="tower_upright_height" value="0.5"/>
+    <xacro:property name="tower_upright_x_size" value="0.02"/>
+    <xacro:property name="tower_upright_y_size" value="0.02"/>
+    <xacro:property name="tower_upright_z_offset" value="${tower_upright_height/2 + chassis_z_size/2}"/>
+    <xacro:property name="camera_size" value="0.05"/>
+    <xacro:property name="camera_roll" value="${pi/4}"/>
+    <xacro:property name="camera_y_offset" value="0.03"/>
+    <xacro:property name="camera_z_offset" value="${tower_upright_height/2}"/>
+    <!-- JOINTS AND LINKS
+         This section uses all the values calculated above to actually create
+         all the links and joints of the robot
+    -->
     <!-- Footprint of the robot (because gazebo's base_link can't have interia) -->
     <link name='base_link'/>
@@ -44,10 +61,17 @@
         <parent link="base_link"/>
         <child link="chassis"/>
+        <origin xyz="
+            ${chassis_x_pos}
+            ${chassis_y_pos}
+            ${chassis_z_pos}
+            "
+            rpy="0 0 0"
+            />
     </joint>
     <box_link
         name="chassis"
-        x_pos="${chassis_x_pos}"
-        y_pos="${chassis_y_pos}"
-        z_pos="${chassis_z_pos}"
+        x_pos="0"
+        y_pos="0"
+        z_pos="0"
         x_size="${chassis_y_size}"
         y_size="${chassis_x_size}"
@@ -64,5 +88,11 @@
             <parent link="chassis"/>
             <child link="${lr_prefix}_primary_rocker"/>
-            <origin xyz="${primary_rocker_x_pos*reflect} ${primary_rocker_y_pos} ${primary_rocker_z_pos}" rpy="0 0 0" />
+            <origin xyz="
+                ${primary_rocker_x_offset*reflect}
+                ${primary_rocker_y_offset}
+                ${primary_rocker_z_offset}
+                "
+                rpy="0 0 0"
+                />
             <axis xyz="1 0 0" rpy="0 0 0" />
             <limit effort="100" velocity="100"/>
@@ -180,3 +210,53 @@
     <primary_wheel lr_prefix="L" fb_prefix="BACK" x_reflect="1" y_reflect="-1"/>
     <primary_wheel lr_prefix="R" fb_prefix="BACK" x_reflect="-1" y_reflect="-1"/>
+    <joint name="chassis_to_tower" type="fixed">
+        <parent link="chassis"/>
+        <child link="tower_upright"/>
+        <origin xyz="
+            0
+            ${tower_upright_y_offset}
+            ${tower_upright_z_offset}
+            "
+            rpy="0 0 0"
+            />
+    </joint>
+    <box_link
+        name="tower_upright"
+        x_pos="0"
+        y_pos="0"
+        z_pos="0"
+        x_size="${tower_upright_x_size}"
+        y_size="${tower_upright_y_size}"
+        z_size="${tower_upright_height}"
+        roll="0"
+        pitch="0"
+        yaw="0"
+        mass="10"
+        material_name="grey"
+        />
+    <joint name="tower_upright_to_camera" type="fixed">
+        <parent link="tower_upright"/>
+        <child link="camera"/>
+        <origin xyz="
+            0
+            ${camera_y_offset}
+            ${camera_z_offset}
+            "
+            rpy="${camera_roll} 0 0"
+            />
+    </joint>
+    <box_link
+        name="camera"
+        x_pos="0"
+        y_pos="0"
+        z_pos="0"
+        x_size="${camera_size}"
+        y_size="${camera_size}"
+        z_size="${camera_size}"
+        roll="0"
+        pitch="0"
+        yaw="0"
+        mass="10"
+        material_name="grey"
+        />
 </robot>

Commit message: Switched x and y in rover_2018 model

File: src/sb_gazebo/robots/rover_2018.xacro (robot description, xacro)
@@ -11,6 +11,6 @@
     <xacro:include filename="$(find sb_gazebo)/robots/materials.xacro"/>
     <xacro:include filename="$(find sb_gazebo)/robots/rover_2018.gazebo"/>
+    <xacro:property name="chassis_x_size" value="0.7"/>
     <xacro:property name="chassis_y_size" value="0.94"/>
-    <xacro:property name="chassis_x_size" value="0.75"/>
     <xacro:property name="chassis_z_size" value="0.4"/>
     <xacro:property name="chassis_mass" value="10"/>
@@ -21,27 +21,30 @@
     <xacro:property name="primary_rocker_radius" value="0.15"/>
     <xacro:property name="primary_rocker_length" value="0.1"/>
-    <xacro:property name="primary_rocker_chassis_clearance" value="0.1"/>
-    <xacro:property name="primary_rocker_x_offset" value="${chassis_x_size/2 + primary_rocker_length/2 + primary_rocker_chassis_clearance}"/>
-    <xacro:property name="primary_rocker_y_offset" value="0"/>
+    <xacro:property name="primary_rocker_chassis_clearance" value="0.02"/>
+    <xacro:property name="primary_rocker_x_offset" value="0"/>
+    <xacro:property name="primary_rocker_y_offset" value="${chassis_x_size/2 + primary_rocker_length/2 + primary_rocker_chassis_clearance}"/>
     <xacro:property name="primary_rocker_z_offset" value="0"/>
     <xacro:property name="primary_rocker_arm_length" value="0.4"/>
     <xacro:property name="primary_rocker_arm_radius" value="0.03"/>
     <xacro:property name="primary_rocker_arm_pitch" value="${pi*2.7/4}"/>
-    <xacro:property name="primary_rocker_arm_x_offset" value="0"/>
-    <xacro:property name="primary_rocker_arm_y_offset" value="${primary_rocker_radius - cos(primary_rocker_arm_pitch)*primary_rocker_arm_length/2}"/>
-    <xacro:property name="primary_rocker_arm_z_offset" value="${- sin(primary_rocker_arm_pitch)*primary_rocker_arm_length/2}"/>
+    <xacro:property name="primary_rocker_arm_x_offset"
+        value="${primary_rocker_radius - cos(primary_rocker_arm_pitch)*primary_rocker_arm_length/2}"
+        />
+    <xacro:property name="primary_rocker_arm_y_offset" value="0"/>
+    <xacro:property name="primary_rocker_arm_z_offset"
+        value="${- sin(primary_rocker_arm_pitch)*primary_rocker_arm_length/2}"/>
     <xacro:property name="primary_wheel_axle_length" value="0.1"/>
     <xacro:property name="primary_wheel_axle_radius" value="0.015"/>
-    <xacro:property name="primary_wheel_axle_x_offset" value="${primary_wheel_axle_length/2}"/>
-    <xacro:property name="primary_wheel_axle_y_offset"
+    <xacro:property name="primary_wheel_axle_x_offset"
         value="${sin(primary_rocker_arm_pitch)*primary_rocker_arm_length/2}"/>
+    <xacro:property name="primary_wheel_axle_y_offset" value="${primary_wheel_axle_length/2}"/>
     <xacro:property name="primary_wheel_axle_z_offset"
         value="${cos(primary_rocker_arm_pitch)*primary_rocker_arm_length/2}"/>
     <xacro:property name="primary_wheel_length" value="0.15"/>
     <xacro:property name="primary_wheel_radius" value="0.17"/>
-    <xacro:property name="primary_wheel_x_offset" value="${primary_wheel_length/2}"/>
-    <xacro:property name="primary_wheel_y_offset" value="0"/>
+    <xacro:property name="primary_wheel_x_offset" value="0"/>
+    <xacro:property name="primary_wheel_y_offset" value="${primary_wheel_length/2}"/>
     <xacro:property name="primary_wheel_z_offset" value="0"/>
-    <xacro:property name="tower_upright_y_offset" value="${chassis_y_size/2}"/>
+    <xacro:property name="tower_upright_x_offset" value="${chassis_y_size/2}"/>
     <xacro:property name="tower_upright_height" value="0.5"/>
     <xacro:property name="tower_upright_x_size" value="0.02"/>
@@ -49,6 +52,6 @@
     <xacro:property name="tower_upright_z_offset" value="${tower_upright_height/2 + chassis_z_size/2}"/>
     <xacro:property name="camera_size" value="0.05"/>
-    <xacro:property name="camera_roll" value="${pi/4}"/>
-    <xacro:property name="camera_y_offset" value="0.03"/>
+    <xacro:property name="camera_pitch" value="${pi/4}"/>
+    <xacro:property name="camera_x_offset" value="0.03"/>
     <xacro:property name="camera_z_offset" value="${tower_upright_height/2}"/>
     <!-- JOINTS AND LINKS
@@ -74,6 +77,6 @@
         y_pos="0"
         z_pos="0"
-        x_size="${chassis_y_size}"
-        y_size="${chassis_x_size}"
+        x_size="${chassis_x_size}"
+        y_size="${chassis_y_size}"
         z_size="${chassis_z_size}"
         roll="0"
@@ -83,5 +86,5 @@
         material_name="grey"
         />
-    <xacro:macro name="primary_rocker" params="lr_prefix reflect">
+    <xacro:macro name="primary_rocker" params="lr_prefix y_reflect">
         <!-- TODO: Make this revolute model with a spring to resist rotation (but allow it) instead of just being fixed like it currently is -->
         <joint name="${lr_prefix}_primary_rocker_to_chassis" type="revolute">
@@ -89,11 +92,15 @@
             <child link="${lr_prefix}_primary_rocker"/>
             <origin xyz="
-                ${primary_rocker_x_offset*reflect}
-                ${primary_rocker_y_offset}
+                ${primary_rocker_x_offset}
+                ${primary_rocker_y_offset*y_reflect}
                 ${primary_rocker_z_offset}
                 "
-                rpy="0 0 0"
+                rpy="
+                0
+                0
+                0
+                "
                 />
-            <axis xyz="1 0 0" rpy="0 0 0" />
+            <axis xyz="0 1 0" rpy="0 0 0" />
             <limit effort="100" velocity="100"/>
             <joint_properties damping="0.0" friction="0.0"/>
@@ -107,5 +114,5 @@
             radius="${primary_rocker_radius}"
             length="${primary_rocker_length}"
-            roll="0"
+            roll="${pi/2}"
             pitch="${pi/2}"
             yaw="0"
@@ -114,6 +121,6 @@
             />
     </xacro:macro>
-    <primary_rocker lr_prefix="L" reflect="1"/>
-    <primary_rocker lr_prefix="R" reflect="-1"/>
+    <primary_rocker lr_prefix="L" y_reflect="1"/>
+    <primary_rocker lr_prefix="R" y_reflect="-1"/>
     <xacro:macro name="primary_rocker_arm" params="lr_prefix fb_prefix x_reflect y_reflect">
         <joint name="${lr_prefix}_${fb_prefix}_primary_rocker_to_primary_rocker_arm" type="fixed">
@@ -136,6 +143,6 @@
             length="${primary_rocker_arm_length}"
             roll="0"
-            pitch="${primary_rocker_arm_pitch*y_reflect}"
-            yaw="${pi/2}"
+            pitch="${primary_rocker_arm_pitch*x_reflect}"
+            yaw="0"
             mass="1"
             material_name="grey"
@@ -143,6 +150,6 @@
     </xacro:macro>
     <primary_rocker_arm lr_prefix="L" fb_prefix="FRONT" x_reflect="1" y_reflect="1"/>
-    <primary_rocker_arm lr_prefix="R" fb_prefix="FRONT" x_reflect="-1" y_reflect="1"/>
-    <primary_rocker_arm lr_prefix="L" fb_prefix="BACK" x_reflect="1" y_reflect="-1"/>
+    <primary_rocker_arm lr_prefix="R" fb_prefix="FRONT" x_reflect="1" y_reflect="-1"/>
+    <primary_rocker_arm lr_prefix="L" fb_prefix="BACK" x_reflect="-1" y_reflect="1"/>
     <primary_rocker_arm lr_prefix="R" fb_prefix="BACK" x_reflect="-1" y_reflect="-1"/>
     <xacro:macro name="primary_wheel_axle" params="lr_prefix fb_prefix x_reflect y_reflect">
@@ -165,5 +172,5 @@
             radius="${primary_wheel_axle_radius}"
             length="${primary_wheel_axle_length}"
-            roll="0"
+            roll="${pi/2}"
             pitch="${pi/2}"
             yaw="0"
@@ -173,9 +180,9 @@
     </xacro:macro>
     <primary_wheel_axle lr_prefix="L" fb_prefix="FRONT" x_reflect="1" y_reflect="1"/>
-    <primary_wheel_axle lr_prefix="R" fb_prefix="FRONT" x_reflect="-1" y_reflect="1"/>
-    <primary_wheel_axle lr_prefix="L" fb_prefix="BACK" x_reflect="1" y_reflect="-1"/>
+    <primary_wheel_axle lr_prefix="R" fb_prefix="FRONT" x_reflect="1" y_reflect="-1"/>
+    <primary_wheel_axle lr_prefix="L" fb_prefix="BACK" x_reflect="-1" y_reflect="1"/>
     <primary_wheel_axle lr_prefix="R" fb_prefix="BACK" x_reflect="-1" y_reflect="-1"/>
     <xacro:macro name="primary_wheel" params="lr_prefix fb_prefix x_reflect y_reflect">
-        <joint name="${lr_prefix}_${fb_prefix}_primary_rocker_arm_to_primary_wheel" type="continuous">
+        <joint name="${lr_prefix}_${fb_prefix}_primary_wheel_axle_to_primary_wheel" type="continuous">
             <parent link="${lr_prefix}_${fb_prefix}_primary_wheel_axle"/>
             <child link="${lr_prefix}_${fb_prefix}_primary_wheel"/>
@@ -187,5 +194,5 @@
                 rpy="0 0 0"
                 />
-            <axis xyz="1 0 0" rpy="0 0 0" />
+            <axis xyz="0 1 0" rpy="0 0 0" />
             <limit effort="100" velocity="100"/>
             <joint_properties damping="0.0" friction="0.0"/>
@@ -199,5 +206,5 @@
             radius="${primary_wheel_radius}"
             length="${primary_wheel_length}"
-            roll="0"
+            roll="${pi/2}"
             pitch="${pi/2}"
             yaw="0"
@@ -207,6 +214,6 @@
     </xacro:macro>
     <primary_wheel lr_prefix="L" fb_prefix="FRONT" x_reflect="1" y_reflect="1"/>
-    <primary_wheel lr_prefix="R" fb_prefix="FRONT" x_reflect="-1" y_reflect="1"/>
-    <primary_wheel lr_prefix="L" fb_prefix="BACK" x_reflect="1" y_reflect="-1"/>
+    <primary_wheel lr_prefix="R" fb_prefix="FRONT" x_reflect="1" y_reflect="-1"/>
+    <primary_wheel lr_prefix="L" fb_prefix="BACK" x_reflect="-1" y_reflect="1"/>
     <primary_wheel lr_prefix="R" fb_prefix="BACK" x_reflect="-1" y_reflect="-1"/>
     <joint name="chassis_to_tower" type="fixed">
@@ -214,6 +221,6 @@
         <child link="tower_upright"/>
         <origin xyz="
+            ${tower_upright_x_offset}
             0
-            ${tower_upright_y_offset}
             ${tower_upright_z_offset}
             "
@@ -239,9 +246,9 @@
         <child link="camera"/>
         <origin xyz="
+            ${camera_x_offset}
             0
-            ${camera_y_offset}
             ${camera_z_offset}
             "
-            rpy="${camera_roll} 0 0"
+            rpy="0 ${camera_pitch} 0"
             />
     </joint>
