Commit message: Very basic rover model

File: src/sb_gazebo/robots/macros.xacro (robot description, xacro)
@@ -4,4 +4,5 @@
 -->
 <robot name="robot" xmlns:xacro="http://www.ros.org/wiki/xacro">
+<!-- Calculate the intertia settings for a cylinder with given mass, radius, height -->
 <xacro:macro name="cylinder_inertia" params="m r h">
   <inertia  ixx="${m*(3*r*r+h*h)/12}" ixy = "0" ixz = "0"
@@ -10,4 +11,5 @@
   />
 </xacro:macro>
+<!-- Calculate the intertia settings for a box with given mass, radius, height -->
 <xacro:macro name="box_inertia" params="m x y z">
   <inertia  ixx="${m*(y*y+z*z)/12}" ixy = "0" ixz = "0"
@@ -16,4 +18,5 @@
   />
 </xacro:macro>
+<!-- Calculate the intertia settings for a sphere with given mass, radius, height -->
 <xacro:macro name="sphere_inertia" params="m r">
   <inertia  ixx="${2*m*r*r/5}" ixy = "0" ixz = "0"
@@ -21,4 +24,56 @@
     izz="${2*m*r*r/5}"
   />
+</xacro:macro>
+<!--
+     Creates a box link
+-->
+<xacro:macro name="box_link"
+    params="name x_pos y_pos z_pos x_size y_size z_size roll pitch yaw mass material_name">
+    <link name="${name}">
+        <collision>
+            <origin xyz="${x_pos} ${y_pos} ${z_pos}" rpy="${roll} ${pitch} ${yaw}"/>
+            <geometry>
+                <box size="${y_size} ${x_size} ${z_size}"/>
+            </geometry>
+        </collision>
+        <visual>
+            <origin xyz="${x_pos} ${y_pos} ${z_pos}" rpy="${roll} ${pitch} ${yaw}"/>
+            <geometry>
+                <box size="${y_size} ${x_size} ${z_size}"/>
+            </geometry>
+            <material name="${material_name}"/>
+        </visual>
+        <inertial>
+            <origin xyz="${x_pos} ${y_pos} ${z_pos}" rpy="${roll} ${pitch} ${yaw}"/>
+            <mass value="${mass}"/>
+            <box_inertia m="${mass}" x="${x_size}" y="${y_size}" z="${z_size}"/>
+        </inertial>
+    </link>
+</xacro:macro>
+<!--
+     Creates a cylinder link
+-->
+<xacro:macro name="cylinder_link"
+    params="name x_pos y_pos z_pos radius length roll pitch yaw mass material_name">
+    <link name="${name}">
+        <collision>
+            <origin xyz="${x_pos} ${y_pos} ${z_pos}" rpy="${roll} ${pitch} ${yaw}"/>
+            <geometry>
+                <cylinder radius="${radius}" length="${length}"/>
+            </geometry>
+        </collision>
+        <visual>
+            <origin xyz="${x_pos} ${y_pos} ${z_pos}" rpy="${roll} ${pitch} ${yaw}"/>
+            <geometry>
+                <cylinder radius="${radius}" length="${length}"/>
+            </geometry>
+            <material name="${material_name}"/>
+        </visual>
+        <inertial>
+            <origin xyz="${x_pos} ${y_pos} ${z_pos}" rpy="${roll} ${pitch} ${yaw}"/>
+            <mass value="${mass}"/>
+            <cylinder_inertia m="${mass}" r="${radius}" h="${length}"/>
+        </inertial>
+    </link>
 </xacro:macro>
 <!-- Macro to generate wheels -->

File: src/sb_gazebo/robots/rover_2018.xacro (robot description, xacro)
@@ -1,2858 +1,154 @@
-<?xml version='1.0'?>
+<?xml version="1.0"?>
 <!--
-     The model for the 2018 "mars" rover
-     This rover has a double roger-bogie suspension design
-     TODO: Conver to use proper constants and macros to reduce duplication
-     TODO: `wheel_hinge_X` -> `wheel_1_axle`
-     TODO: Rename joints to be more descriptive
+     The Model for elsa-x, a 2-wheel drive robot with front and back caster wheels
 -->
 <robot name="rover_2018" xmlns:xacro="http://www.ros.org/wiki/xacro">
+    <xacro:include filename="$(find sb_gazebo)/robots/macros.xacro"/>
+    <xacro:include filename="$(find sb_gazebo)/robots/materials.xacro"/>
+    <xacro:include filename="$(find sb_gazebo)/robots/rover_2018.gazebo"/>
+    <xacro:property name="chassis_y_size" value="0.94"/>
+    <xacro:property name="chassis_x_size" value="0.75"/>
+    <xacro:property name="chassis_z_size" value="0.4"/>
+    <xacro:property name="chassis_mass" value="10"/>
+    <xacro:property name="chassis_elevation" value="0.5"/>
+    <xacro:property name="chassis_x_pos" value="0"/>
+    <xacro:property name="chassis_y_pos" value="0"/>
+    <xacro:property name="chassis_z_pos" value="${chassis_z_size + chassis_elevation}"/>
+    <xacro:property name="primary_rocker_radius" value="0.15"/>
+    <xacro:property name="primary_rocker_length" value="0.1"/>
+    <xacro:property name="primary_rocker_chassis_clearance" value="0.1"/>
+    <xacro:property name="primary_rocker_x_pos" value="${chassis_x_size/2 + primary_rocker_length/2 + primary_rocker_chassis_clearance}"/>
+    <xacro:property name="primary_rocker_y_pos" value="0"/>
+    <xacro:property name="primary_rocker_z_pos" value="${chassis_z_size + chassis_elevation}"/>
+    <xacro:property name="primary_rocker_arm_length" value="0.4"/>
+    <xacro:property name="primary_rocker_arm_radius" value="0.03"/>
+    <xacro:property name="primary_rocker_arm_pitch" value="${pi*2.7/4}"/>
+    <xacro:property name="primary_rocker_arm_x_pos" value="${primary_rocker_x_pos}"/>
+    <xacro:property name="primary_rocker_arm_y_pos" value="${primary_rocker_radius - cos(primary_rocker_arm_pitch)*primary_rocker_arm_length/2}"/>
+    <xacro:property name="primary_rocker_arm_z_pos" value="${chassis_z_size + chassis_elevation - sin(primary_rocker_arm_pitch)*primary_rocker_arm_length/2}"/>
+    <xacro:property name="primary_wheel_axle_length" value="0.1"/>
+    <xacro:property name="primary_wheel_axle_radius" value="0.015"/>
+    <xacro:property name="primary_wheel_axle_x_pos" value="${primary_rocker_x_pos}"/>
+    <xacro:property name="primary_wheel_axle_y_pos" value="${primary_rocker_y_pos + cos(primary_rocker_arm_pitch)*primary_rocker_arm_length*2}"/>
+    <xacro:property name="primary_wheel_axle_z_pos" value="${primary_rocker_arm_z_pos - sin(primary_rocker_arm_pitch)*primary_rocker_arm_length/2}"/>
+    <xacro:property name="primary_wheel_length" value="0.15"/>
+    <xacro:property name="primary_wheel_radius" value="0.17"/>
+    <xacro:property name="primary_wheel_x_pos" value="${primary_wheel_axle_x_pos + primary_wheel_axle_length/2 + primary_wheel_length/2}"/>
+    <xacro:property name="primary_wheel_y_pos" value="${primary_wheel_axle_y_pos}"/>
+    <xacro:property name="primary_wheel_z_pos" value="${primary_wheel_axle_z_pos}"/>
     <!-- Footprint of the robot (because gazebo's base_link can't have interia) -->
     <link name='base_link'/>
     <joint name="base_joint" type="fixed">
         <parent link="base_link"/>
-        <child link="main_chassis"/>
+        <child link="chassis"/>
     </joint>
-    <link name='main_chassis'>
-        <pose frame=''>-0.495954 0.481744 0.172621 0 -0 0</pose>
-        <inertial>
-            <mass value="10"/>
-            <inertia
-                ixx="0.01"
-                ixy="0"
-                ixz="0"
-                iyy="0.01"
-                iyz="0"
-                izz="0.01"
+    <box_link
+        name="chassis"
+        x_pos="${chassis_x_pos}"
+        y_pos="${chassis_y_pos}"
+        z_pos="${chassis_z_pos}"
+        x_size="${chassis_y_size}"
+        y_size="${chassis_x_size}"
+        z_size="${chassis_z_size}"
+        roll="0"
+        pitch="0"
+        yaw="0"
+        mass="10"
+        material_name="grey"
+        />
+    <xacro:macro name="primary_rocker" params="lr_prefix reflect">
+        <joint name="${lr_prefix}_primary_rocker_to_chassis" type="fixed">
+            <parent link="chassis"/>
+            <child link="${lr_prefix}_primary_rocker"/>
+        </joint>
+        <cylinder_link
+            name="${lr_prefix}_primary_rocker"
+            x_pos="${primary_rocker_x_pos*reflect}"
+            y_pos="${primary_rocker_y_pos}"
+            z_pos="${primary_rocker_z_pos}"
+            radius="${primary_rocker_radius}"
+            length="${primary_rocker_length}"
+            roll="0"
+            pitch="${pi/2}"
+            yaw="0"
+            mass="1"
+            material_name="grey"
             />
-            <pose frame=''>0 0 0 0 -0 0</pose>
-        </inertial>
-        <self_collide>0</self_collide>
-        <kinematic>0</kinematic>
-        <enable_wind>0</enable_wind>
-        <visual name='visual'>
-            <pose frame=''>0 0 0 0 -0 0</pose>
-            <geometry>
-                <box
-                    size="1.09569 1.7415 0.312322"
-                />
-            </geometry>
-            <material name="grey">
-                <lighting>1</lighting>
-                <script>
-                    <uri>file://media/materials/scripts/gazebo.material</uri>
-                    <name>Gazebo/Grey</name>
-                </script>
-                <ambient>0.3 0.3 0.3 1</ambient>
-                <diffuse>0.7 0.7 0.7 1</diffuse>
-                <specular>0.01 0.01 0.01 1</specular>
-                <emissive>0 0 0 1</emissive>
-                <shader type='vertex'>
-                    <normal_map>__default__</normal_map>
-                </shader>
-            </material>
-            <cast_shadows>1</cast_shadows>
-            <transparency>0</transparency>
-        </visual>
-        <collision name='collision'>
-            <laser_retro>0</laser_retro>
-            <max_contacts>10</max_contacts>
-            <pose frame=''>0 0 0 0 -0 0</pose>
-            <geometry>
-                <box
-                    size="1.09569 1.7415 0.312322"
-                />
-            </geometry>
-            <surface>
-                <friction>
-                    <ode>
-                        <mu>1</mu>
-                        <mu2>1</mu2>
-                        <fdir1>0 0 0</fdir1>
-                        <slip1>0</slip1>
-                        <slip2>0</slip2>
-                    </ode>
-                    <torsional>
-                        <coefficient>1</coefficient>
-                        <patch_radius>0</patch_radius>
-                        <surface_radius>0</surface_radius>
-                        <use_patch_radius>1</use_patch_radius>
-                        <ode>
-                            <slip>0</slip>
-                        </ode>
-                    </torsional>
-                </friction>
-                <bounce>
-                    <restitution_coefficient>0</restitution_coefficient>
-                    <threshold>1e+06</threshold>
-                </bounce>
-                <contact>
-                    <collide_without_contact>0</collide_without_contact>
-                    <collide_without_contact_bitmask>1</collide_without_contact_bitmask>
-                    <collide_bitmask>1</collide_bitmask>
-                    <ode>
-                        <soft_cfm>0</soft_cfm>
-                        <soft_erp>0.2</soft_erp>
-                        <kp>1e+13</kp>
-                        <kd>1</kd>
-                        <max_vel>0.01</max_vel>
-                        <min_depth>0</min_depth>
-                    </ode>
-                    <bullet>
-                        <split_impulse>1</split_impulse>
-                        <split_impulse_penetration_threshold>-0.01</split_impulse_penetration_threshold>
-                        <soft_cfm>0</soft_cfm>
-                        <soft_erp>0.2</soft_erp>
-                        <kp>1e+13</kp>
-                        <kd>1</kd>
-                    </bullet>
-                </contact>
-            </surface>
-        </collision>
-    </link>
-    <link name='L_primary_rocker'>
-        <pose frame=''>0.120732 0.480291 0.210888 3.14159 -1.57 -3.14159</pose>
-        <inertial>
-            <mass value="0.0046174"/>
-            <inertia
-                ixx="0.01"
-                ixy="0"
-                ixz="0"
-                iyy="0.01"
-                iyz="0"
-                izz="0.01"
+    </xacro:macro>
+    <primary_rocker lr_prefix="L" reflect="1"/>
+    <primary_rocker lr_prefix="R" reflect="-1"/>
+    <xacro:macro name="primary_rocker_arm" params="lr_prefix fb_prefix x_reflect y_reflect">
+        <joint name="${lr_prefix}_${fb_prefix}_primary_rocker_to_primary_rocker_arm" type="fixed">
+            <parent link="${lr_prefix}_primary_rocker"/>
+            <child link="${lr_prefix}_${fb_prefix}_primary_rocker_arm"/>
+        </joint>
+        <cylinder_link
+            name="${lr_prefix}_${fb_prefix}_primary_rocker_arm"
+            x_pos="${primary_rocker_arm_x_pos*x_reflect}"
+            y_pos="${primary_rocker_arm_y_pos*y_reflect}"
+            z_pos="${primary_rocker_arm_z_pos}"
+            radius="${primary_rocker_arm_radius}"
+            length="${primary_rocker_arm_length}"
+            roll="0"
+            pitch="${primary_rocker_arm_pitch*y_reflect}"
+            yaw="${pi/2}"
+            mass="1"
+            material_name="grey"
             />
-            <pose frame=''>0 0 0 0 -0 0</pose>
-        </inertial>
-        <self_collide>0</self_collide>
-        <kinematic>0</kinematic>
-        <enable_wind>0</enable_wind>
-        <visual name='visual'>
-            <pose frame=''>0 0 0 0 -0 0</pose>
-            <geometry>
-                <cylinder
-                    radius="0.0992866"
-                    length="0.116478"
-                />
-            </geometry>
-            <material name="grey">
-                <lighting>1</lighting>
-                <script>
-                    <uri>file://media/materials/scripts/gazebo.material</uri>
-                    <name>Gazebo/Grey</name>
-                </script>
-                <ambient>0.3 0.3 0.3 1</ambient>
-                <diffuse>0.7 0.7 0.7 1</diffuse>
-                <specular>0.01 0.01 0.01 1</specular>
-                <emissive>0 0 0 1</emissive>
-                <shader type='vertex'>
-                    <normal_map>__default__</normal_map>
-                </shader>
-            </material>
-            <cast_shadows>1</cast_shadows>
-            <transparency>0</transparency>
-        </visual>
-    </link>
-    <link name='L_primary_rocker_hinge'>
-        <pose frame=''>0.045335 0.475634 0.210685 3.14159 -1.57 -3.14159</pose>
-        <inertial>
-            <mass value="0.00110726"/>
-            <inertia
-                ixx="0.01"
-                ixy="0"
-                ixz="0"
-                iyy="0.01"
-                iyz="0"
-                izz="0.01"
+    </xacro:macro>
+    <primary_rocker_arm lr_prefix="L" fb_prefix="FRONT" x_reflect="1" y_reflect="1"/>
+    <primary_rocker_arm lr_prefix="R" fb_prefix="FRONT" x_reflect="-1" y_reflect="1"/>
+    <primary_rocker_arm lr_prefix="L" fb_prefix="BACK" x_reflect="1" y_reflect="-1"/>
+    <primary_rocker_arm lr_prefix="R" fb_prefix="BACK" x_reflect="-1" y_reflect="-1"/>
+    <xacro:macro name="primary_wheel_axle" params="lr_prefix fb_prefix x_reflect y_reflect">
+        <joint name="${lr_prefix}_${fb_prefix}_primary_rocker_arm_to_primary_wheel_axle" type="fixed">
+            <parent link="${lr_prefix}_${fb_prefix}_primary_rocker_arm"/>
+            <child link="${lr_prefix}_${fb_prefix}_primary_wheel_axle"/>
+        </joint>
+        <cylinder_link
+            name="${lr_prefix}_${fb_prefix}_primary_wheel_axle"
+            x_pos="${(primary_wheel_axle_x_pos + primary_wheel_axle_length/2)*x_reflect}"
+            y_pos="${primary_wheel_axle_y_pos*y_reflect}"
+            z_pos="${primary_wheel_axle_z_pos}"
+            radius="${primary_wheel_axle_radius}"
+            length="${primary_wheel_axle_length}"
+            roll="0"
+            pitch="${pi/2}"
+            yaw="0"
+            mass="0.05"
+            material_name="grey"
             />
-            <pose frame=''>0 0 0 0 -0 0</pose>
-        </inertial>
-        <self_collide>0</self_collide>
-        <kinematic>0</kinematic>
-        <enable_wind>0</enable_wind>
-        <visual name='visual'>
-            <pose frame=''>0 0 0 0 -0 0</pose>
-            <geometry>
-                <cylinder
-                    radius="0.0379471"
-                    length="0.191181"
-                />
-            </geometry>
-            <material name="grey">
-                <lighting>1</lighting>
-                <script>
-                    <uri>file://media/materials/scripts/gazebo.material</uri>
-                    <name>Gazebo/Grey</name>
-                </script>
-                <ambient>0.3 0.3 0.3 1</ambient>
-                <diffuse>0.7 0.7 0.7 1</diffuse>
-                <specular>0.01 0.01 0.01 1</specular>
-                <emissive>0 0 0 1</emissive>
-                <shader type='vertex'>
-                    <normal_map>__default__</normal_map>
-                </shader>
-            </material>
-            <cast_shadows>1</cast_shadows>
-            <transparency>0</transparency>
-        </visual>
-    </link>
-    <link name='L_primary_wheel_arm_backwards'>
-        <pose frame=''>0.120732 0.773902 0.074463 -0.422885 0 0</pose>
-        <inertial>
-            <mass value="0.00541225"/>
-            <inertia
-                ixx="0.01"
-                ixy="0"
-                ixz="0"
-                iyy="0.01"
-                iyz="0"
-                izz="0.01"
+    </xacro:macro>
+    <primary_wheel_axle lr_prefix="L" fb_prefix="FRONT" x_reflect="1" y_reflect="1"/>
+    <primary_wheel_axle lr_prefix="R" fb_prefix="FRONT" x_reflect="-1" y_reflect="1"/>
+    <primary_wheel_axle lr_prefix="L" fb_prefix="BACK" x_reflect="1" y_reflect="-1"/>
+    <primary_wheel_axle lr_prefix="R" fb_prefix="BACK" x_reflect="-1" y_reflect="-1"/>
+    <xacro:macro name="primary_wheel" params="lr_prefix fb_prefix x_reflect y_reflect">
+        <joint name="${lr_prefix}_${fb_prefix}_primary_rocker_arm_to_primary_wheel" type="continuous">
+            <parent link="${lr_prefix}_${fb_prefix}_primary_rocker_arm"/>
+            <child link="${lr_prefix}_${fb_prefix}_primary_wheel"/>
+            <origin xyz="${primary_wheel_x_pos*x_reflect} ${primary_wheel_y_pos*y_reflect} ${primary_wheel_z_pos}" rpy="0 0 0" />
+            <axis xyz="1 0 0" rpy="0 0 0" />
+            <limit effort="100" velocity="100"/>
+            <joint_properties damping="0.0" friction="0.0"/>
+            <hardwareInterface>EffortJointInterface</hardwareInterface>
+        </joint>
+        <cylinder_link
+            name="${lr_prefix}_${fb_prefix}_primary_wheel"
+            x_pos="0"
+            y_pos="0"
+            z_pos="0"
+            radius="${primary_wheel_radius}"
+            length="${primary_wheel_length}"
+            roll="0"
+            pitch="${pi/2}"
+            yaw="0"
+            mass="1"
+            material_name="grey"
             />
-            <pose frame=''>0 0 0 0 -0 0</pose>
-        </inertial>
-        <self_collide>0</self_collide>
-        <kinematic>0</kinematic>
-        <enable_wind>0</enable_wind>
-        <gravity>1</gravity>
-        <visual name='visual'>
-            <pose frame=''>0 0 0 0 -0 0</pose>
-            <geometry>
-                <box
-                    size="0.093481 0.512407 0.11302"
-                />
-            </geometry>
-            <material name="grey">
-                <lighting>1</lighting>
-                <script>
-                    <uri>file://media/materials/scripts/gazebo.material</uri>
-                    <name>Gazebo/Grey</name>
-                </script>
-                <ambient>0.3 0.3 0.3 1</ambient>
-                <diffuse>0.7 0.7 0.7 1</diffuse>
-                <specular>0.01 0.01 0.01 1</specular>
-                <emissive>0 0 0 1</emissive>
-                <shader type='pixel'>
-                    <normal_map>__default__</normal_map>
-                </shader>
-            </material>
-            <cast_shadows>1</cast_shadows>
-            <transparency>0</transparency>
-        </visual>
-        <collision name='collision'>
-            <laser_retro>0</laser_retro>
-            <max_contacts>10</max_contacts>
-            <pose frame=''>0 0 0 0 -0 0</pose>
-            <geometry>
-                <box
-                    size="0.093481 0.512407 0.11302"
-                />
-            </geometry>
-            <surface>
-                <friction>
-                    <ode>
-                        <mu>1</mu>
-                        <mu2>1</mu2>
-                        <fdir1>0 0 0</fdir1>
-                        <slip1>0</slip1>
-                        <slip2>0</slip2>
-                    </ode>
-                    <torsional>
-                        <coefficient>1</coefficient>
-                        <patch_radius>0</patch_radius>
-                        <surface_radius>0</surface_radius>
-                        <use_patch_radius>1</use_patch_radius>
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