Commit message: Addressed PR comments (mostly documentation)

File: src/sb_gazebo/robots/macros.xacro (robot description, xacro)
@@ -11,5 +11,5 @@
   />
 </xacro:macro>
-<!-- Calculate the intertia settings for a box with given mass, radius, height -->
+<!-- Calculate the intertia settings for a box with given mass, x size, y size, z size -->
 <xacro:macro name="box_inertia" params="m x y z">
   <inertia  ixx="${m*(y*y+z*z)/12}" ixy = "0" ixz = "0"
@@ -18,5 +18,5 @@
   />
 </xacro:macro>
-<!-- Calculate the intertia settings for a sphere with given mass, radius, height -->
+<!-- Calculate the intertia settings for a sphere with given mass, radius -->
 <xacro:macro name="sphere_inertia" params="m r">
   <inertia  ixx="${2*m*r*r/5}" ixy = "0" ixz = "0"

File: src/sb_gazebo/robots/rover_2018.xacro (robot description, xacro)
@@ -21,5 +21,7 @@
     <xacro:property name="primary_rocker_radius" value="0.15"/>
     <xacro:property name="primary_rocker_length" value="0.1"/>
+    <!-- The size of the gap between the chassis and the primary rocker -->
     <xacro:property name="primary_rocker_chassis_clearance" value="0.02"/>
+    <!-- Primary rocker offset from it's parent joint (the chassis) -->
     <xacro:property name="primary_rocker_x_offset" value="0"/>
     <xacro:property name="primary_rocker_y_offset" value="${chassis_x_size/2 + primary_rocker_length/2 + primary_rocker_chassis_clearance}"/>
@@ -86,9 +88,17 @@
         material_name="grey"
         />
-    <xacro:macro name="primary_rocker" params="lr_prefix y_reflect">
+    <!--
+         This macro generates the primary rocker joint between the rocker
+         arms and the main chassis
+         @param left_right_prefix A prefix (should be "left" or "right") that
+         is placed in front of the joint and link name
+         @param y_reflect A value (should be `1` or `-1`) that the y coordinates
+         of the generated joint and link are multiplied by
+    -->
+    <xacro:macro name="primary_rocker" params="left_right_prefix y_reflect">
         <!-- TODO: Make this revolute model with a spring to resist rotation (but allow it) instead of just being fixed like it currently is -->
-        <joint name="${lr_prefix}_primary_rocker_to_chassis" type="revolute">
+        <joint name="${left_right_prefix}_primary_rocker_to_chassis" type="revolute">
             <parent link="chassis"/>
-            <child link="${lr_prefix}_primary_rocker"/>
+            <child link="${left_right_prefix}_primary_rocker"/>
             <origin xyz="
                 ${primary_rocker_x_offset}
@@ -108,5 +118,5 @@
         </joint>
         <cylinder_link
-            name="${lr_prefix}_primary_rocker"
+            name="${left_right_prefix}_primary_rocker"
             x_pos="0"
             y_pos="0"
@@ -121,10 +131,22 @@
             />
     </xacro:macro>
-    <primary_rocker lr_prefix="L" y_reflect="1"/>
-    <primary_rocker lr_prefix="R" y_reflect="-1"/>
-    <xacro:macro name="primary_rocker_arm" params="lr_prefix fb_prefix x_reflect y_reflect">
-        <joint name="${lr_prefix}_${fb_prefix}_primary_rocker_to_primary_rocker_arm" type="fixed">
-            <parent link="${lr_prefix}_primary_rocker"/>
-            <child link="${lr_prefix}_${fb_prefix}_primary_rocker_arm"/>
+    <primary_rocker left_right_prefix="left" y_reflect="1"/>
+    <primary_rocker left_right_prefix="right" y_reflect="-1"/>
+    <!--
+         This macro generates the primary rocker arm between the primary rocker
+         joint and the wheel axles
+         @param left_right_prefix A prefix (should be "left" or "right") that
+         is placed in front of the joint and link name
+         @param front_back_prefix A prefix (should be "front" or "back") that
+         is placed in front of the joint and link name
+         @param y_reflect A value (should be `1` or `-1`) that the y coordinates
+         of the generated joint and link are multiplied by
+         @param y_reflect A value (should be `1` or `-1`) that the x coordinates
+         of the generated joint and link are multiplied by
+    -->
+    <xacro:macro name="primary_rocker_arm" params="left_right_prefix front_back_prefix x_reflect y_reflect">
+        <joint name="${left_right_prefix}_${front_back_prefix}_primary_rocker_to_primary_rocker_arm" type="fixed">
+            <parent link="${left_right_prefix}_primary_rocker"/>
+            <child link="${left_right_prefix}_${front_back_prefix}_primary_rocker_arm"/>
             <origin xyz="
                 ${primary_rocker_arm_x_offset*x_reflect}
@@ -136,5 +158,5 @@
         </joint>
         <cylinder_link
-            name="${lr_prefix}_${fb_prefix}_primary_rocker_arm"
+            name="${left_right_prefix}_${front_back_prefix}_primary_rocker_arm"
             x_pos="0"
             y_pos="0"
@@ -149,12 +171,23 @@
             />
     </xacro:macro>
-    <primary_rocker_arm lr_prefix="L" fb_prefix="FRONT" x_reflect="1" y_reflect="1"/>
-    <primary_rocker_arm lr_prefix="R" fb_prefix="FRONT" x_reflect="1" y_reflect="-1"/>
-    <primary_rocker_arm lr_prefix="L" fb_prefix="BACK" x_reflect="-1" y_reflect="1"/>
-    <primary_rocker_arm lr_prefix="R" fb_prefix="BACK" x_reflect="-1" y_reflect="-1"/>
-    <xacro:macro name="primary_wheel_axle" params="lr_prefix fb_prefix x_reflect y_reflect">
-        <joint name="${lr_prefix}_${fb_prefix}_primary_rocker_arm_to_primary_wheel_axle" type="fixed">
-            <parent link="${lr_prefix}_${fb_prefix}_primary_rocker_arm"/>
-            <child link="${lr_prefix}_${fb_prefix}_primary_wheel_axle"/>
+    <primary_rocker_arm left_right_prefix="left" front_back_prefix="FRONT" x_reflect="1" y_reflect="1"/>
+    <primary_rocker_arm left_right_prefix="right" front_back_prefix="FRONT" x_reflect="1" y_reflect="-1"/>
+    <primary_rocker_arm left_right_prefix="left" front_back_prefix="BACK" x_reflect="-1" y_reflect="1"/>
+    <primary_rocker_arm left_right_prefix="right" front_back_prefix="BACK" x_reflect="-1" y_reflect="-1"/>
+    <!--
+         This macro generates the axle for the primary wheels
+         @param left_right_prefix A prefix (should be "left" or "right") that
+         is placed in front of the joint and link name
+         @param front_back_prefix A prefix (should be "front" or "back") that
+         is placed in front of the joint and link name
+         @param y_reflect A value (should be `1` or `-1`) that the y coordinates
+         of the generated joint and link are multiplied by
+         @param y_reflect A value (should be `1` or `-1`) that the x coordinates
+         of the generated joint and link are multiplied by
+    -->
+    <xacro:macro name="primary_wheel_axle" params="left_right_prefix front_back_prefix x_reflect y_reflect">
+        <joint name="${left_right_prefix}_${front_back_prefix}_primary_rocker_arm_to_primary_wheel_axle" type="fixed">
+            <parent link="${left_right_prefix}_${front_back_prefix}_primary_rocker_arm"/>
+            <child link="${left_right_prefix}_${front_back_prefix}_primary_wheel_axle"/>
             <origin xyz="
                 ${primary_wheel_axle_x_offset*x_reflect}
@@ -166,5 +199,5 @@
         </joint>
         <cylinder_link
-            name="${lr_prefix}_${fb_prefix}_primary_wheel_axle"
+            name="${left_right_prefix}_${front_back_prefix}_primary_wheel_axle"
             x_pos="0"
             y_pos="0"
@@ -179,12 +212,23 @@
             />
     </xacro:macro>
-    <primary_wheel_axle lr_prefix="L" fb_prefix="FRONT" x_reflect="1" y_reflect="1"/>
-    <primary_wheel_axle lr_prefix="R" fb_prefix="FRONT" x_reflect="1" y_reflect="-1"/>
-    <primary_wheel_axle lr_prefix="L" fb_prefix="BACK" x_reflect="-1" y_reflect="1"/>
-    <primary_wheel_axle lr_prefix="R" fb_prefix="BACK" x_reflect="-1" y_reflect="-1"/>
-    <xacro:macro name="primary_wheel" params="lr_prefix fb_prefix x_reflect y_reflect">
-        <joint name="${lr_prefix}_${fb_prefix}_primary_wheel_axle_to_primary_wheel" type="continuous">
-            <parent link="${lr_prefix}_${fb_prefix}_primary_wheel_axle"/>
-            <child link="${lr_prefix}_${fb_prefix}_primary_wheel"/>
+    <primary_wheel_axle left_right_prefix="left" front_back_prefix="FRONT" x_reflect="1" y_reflect="1"/>
+    <primary_wheel_axle left_right_prefix="right" front_back_prefix="FRONT" x_reflect="1" y_reflect="-1"/>
+    <primary_wheel_axle left_right_prefix="left" front_back_prefix="BACK" x_reflect="-1" y_reflect="1"/>
+    <primary_wheel_axle left_right_prefix="right" front_back_prefix="BACK" x_reflect="-1" y_reflect="-1"/>
+    <!--
+         This macro generates the primary wheels
+         @param left_right_prefix A prefix (should be "left" or "right") that
+         is placed in front of the joint and link name
+         @param front_back_prefix A prefix (should be "front" or "back") that
+         is placed in front of the joint and link name
+         @param y_reflect A value (should be `1` or `-1`) that the y coordinates
+         of the generated joint and link are multiplied by
+         @param y_reflect A value (should be `1` or `-1`) that the x coordinates
+         of the generated joint and link are multiplied by
+    -->
+    <xacro:macro name="primary_wheel" params="left_right_prefix front_back_prefix x_reflect y_reflect">
+        <joint name="${left_right_prefix}_${front_back_prefix}_primary_wheel_axle_to_primary_wheel" type="continuous">
+            <parent link="${left_right_prefix}_${front_back_prefix}_primary_wheel_axle"/>
+            <child link="${left_right_prefix}_${front_back_prefix}_primary_wheel"/>
             <origin xyz="
                 ${primary_wheel_x_offset*x_reflect}
@@ -200,5 +244,5 @@
         </joint>
         <cylinder_link
-            name="${lr_prefix}_${fb_prefix}_primary_wheel"
+            name="${left_right_prefix}_${front_back_prefix}_primary_wheel"
             x_pos="0"
             y_pos="0"
@@ -213,8 +257,8 @@
             />
     </xacro:macro>
-    <primary_wheel lr_prefix="L" fb_prefix="FRONT" x_reflect="1" y_reflect="1"/>
-    <primary_wheel lr_prefix="R" fb_prefix="FRONT" x_reflect="1" y_reflect="-1"/>
-    <primary_wheel lr_prefix="L" fb_prefix="BACK" x_reflect="-1" y_reflect="1"/>
-    <primary_wheel lr_prefix="R" fb_prefix="BACK" x_reflect="-1" y_reflect="-1"/>
+    <primary_wheel left_right_prefix="left" front_back_prefix="FRONT" x_reflect="1" y_reflect="1"/>
+    <primary_wheel left_right_prefix="right" front_back_prefix="FRONT" x_reflect="1" y_reflect="-1"/>
+    <primary_wheel left_right_prefix="left" front_back_prefix="BACK" x_reflect="-1" y_reflect="1"/>
+    <primary_wheel left_right_prefix="right" front_back_prefix="BACK" x_reflect="-1" y_reflect="-1"/>
     <joint name="chassis_to_tower" type="fixed">
         <parent link="chassis"/>

Commit message: Rover 2018 Model (#369)
* Created the Initial Rover With Some Broken Physics

* Updated Gazebo Resource Paths In Setup Scripts'

* Moved Files Around To Make Gazebo Happy

* Moved Rover To Models Folder

* Fixed Inertia Matrices So The Robot No Longer Explodes

* Moved Robots to robots FOlder

* Changed Robot Paths In .xacro Files

* Revamped Gazebo Launch File System

* Removed unused launch file

* Added some more dependecies to sb_gazebo package.xml

* Added basic controllers for rover_2018

* Updating Rover Model To Be Xacro compatible

* Added launch file for basic rover course'

* Refactored Launch Files So load_robot.launch is more standalone

* Moved world_path construction to load_world.launch

* Very basic rover model

* Revised Rover Model To Use Relative Positions

* Added Tower And Camera To Rover 2018 Model

* Switched x and y in rover_2018 model

* Added Stereo Camera To rover_2018

* Removed Unused Sections of rover_2018_control.yaml

* Addressed PR comments (mostly documentation)

* Updated travis script to properly fail on non-zero exit codes

* Fixed sb_gazebo package.xml

File: src/sb_gazebo/robots/macros.xacro (robot description, xacro)
@@ -4,4 +4,5 @@
 -->
 <robot name="robot" xmlns:xacro="http://www.ros.org/wiki/xacro">
+<!-- Calculate the intertia settings for a cylinder with given mass, radius, height -->
 <xacro:macro name="cylinder_inertia" params="m r h">
   <inertia  ixx="${m*(3*r*r+h*h)/12}" ixy = "0" ixz = "0"
@@ -10,4 +11,5 @@
   />
 </xacro:macro>
+<!-- Calculate the intertia settings for a box with given mass, x size, y size, z size -->
 <xacro:macro name="box_inertia" params="m x y z">
   <inertia  ixx="${m*(y*y+z*z)/12}" ixy = "0" ixz = "0"
@@ -16,4 +18,5 @@
   />
 </xacro:macro>
+<!-- Calculate the intertia settings for a sphere with given mass, radius -->
 <xacro:macro name="sphere_inertia" params="m r">
   <inertia  ixx="${2*m*r*r/5}" ixy = "0" ixz = "0"
@@ -21,4 +24,56 @@
     izz="${2*m*r*r/5}"
   />
+</xacro:macro>
+<!--
+     Creates a box link
+-->
+<xacro:macro name="box_link"
+    params="name x_pos y_pos z_pos x_size y_size z_size roll pitch yaw mass material_name">
+    <link name="${name}">
+        <collision>
+            <origin xyz="${x_pos} ${y_pos} ${z_pos}" rpy="${roll} ${pitch} ${yaw}"/>
+            <geometry>
+                <box size="${y_size} ${x_size} ${z_size}"/>
+            </geometry>
+        </collision>
+        <visual>
+            <origin xyz="${x_pos} ${y_pos} ${z_pos}" rpy="${roll} ${pitch} ${yaw}"/>
+            <geometry>
+                <box size="${y_size} ${x_size} ${z_size}"/>
+            </geometry>
+            <material name="${material_name}"/>
+        </visual>
+        <inertial>
+            <origin xyz="${x_pos} ${y_pos} ${z_pos}" rpy="${roll} ${pitch} ${yaw}"/>
+            <mass value="${mass}"/>
+            <box_inertia m="${mass}" x="${x_size}" y="${y_size}" z="${z_size}"/>
+        </inertial>
+    </link>
+</xacro:macro>
+<!--
+     Creates a cylinder link
+-->
+<xacro:macro name="cylinder_link"
+    params="name x_pos y_pos z_pos radius length roll pitch yaw mass material_name">
+    <link name="${name}">
+        <collision>
+            <origin xyz="${x_pos} ${y_pos} ${z_pos}" rpy="${roll} ${pitch} ${yaw}"/>
+            <geometry>
+                <cylinder radius="${radius}" length="${length}"/>
+            </geometry>
+        </collision>
+        <visual>
+            <origin xyz="${x_pos} ${y_pos} ${z_pos}" rpy="${roll} ${pitch} ${yaw}"/>
+            <geometry>
+                <cylinder radius="${radius}" length="${length}"/>
+            </geometry>
+            <material name="${material_name}"/>
+        </visual>
+        <inertial>
+            <origin xyz="${x_pos} ${y_pos} ${z_pos}" rpy="${roll} ${pitch} ${yaw}"/>
+            <mass value="${mass}"/>
+            <cylinder_inertia m="${mass}" r="${radius}" h="${length}"/>
+        </inertial>
+    </link>
 </xacro:macro>
 <!-- Macro to generate wheels -->
