Commit message: New configs for Noetic

File: src/snowbots_arm_urdf_simplified_v5_12/urdf/snowbots_arm_urdf_simplified_v5_12.urdf (robot description, URDF)
Before this commit: robot snowbots_arm_urdf_simplified_v5_12, 8 links, 7 joints
Links:
- added link world; visual mesh filename=package://snowbots_arm_urdf_simplified_v5_12/meshes/l1.STL
Joints:
- added joint fixer: type fixed, parent world, child l1, origin xyz=0 0 0 rpy=0 0 0, axis 0 0 0
